File: BedStrip.sch (EAGLE design)
At the start: 25 parts, among them IC1 74AHCT2G125DP,125, IC4 LM2596S

Commit message: Ready for PCB MFG
Parts:
- renumbered MOTION to PIR.SENSOR
Connections:
- net 3.3V renamed VCC_3V3.2
- new net VCC_3V3.1: U$1.3.3V@2
- new net VCC_3V3.3: U$1.3.3V@5
- net 12V: now also POWER.1; no longer POWER.2
- net 5V: now also 5V_LED.1, U$1.VIN; no longer 5V_LED.3, U$1.VV
- net GND: now also 5V_LED.3, POWER.2; no longer 5V_LED.1, POWER.1
Other:
- moved on the sheet: 5V_LED, POWER
Changed lines of the file:
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@@
 <clearance class="1" value="0.127"/>
 </class>
-<class number="2" name="signal" width="0.1524" drill="0">
+<class number="2" name="signal" width="0.002540625" drill="0">
 <clearance class="2" value="0.0508"/>
 </class>
-<class number="3" name="HV" width="0.508" drill="0">
+<class number="3" name="HV" width="0.254" drill="0">
 <clearance class="3" value="0.127"/>
 </class>
@@
 <part name="SUPPLY15" library="supply2" library_urn="urn:adsk.eagle:library:372" deviceset="GND" device=""/>
 <part name="SUPPLY12" library="supply2" library_urn="urn:adsk.eagle:library:372" deviceset="GND" device=""/>
-<part name="U$1" library="CustomParts-Josh" library_urn="urn:adsk.eagle:library:21718240" deviceset="DEVBOARD_ESP8266_NODEMCU_V3" device="DEVBOARD" package3d_urn="urn:adsk.eagle:package:36294322/3"/>
+<part name="U$1" library="CustomParts-Josh" library_urn="urn:adsk.eagle:library:21718240" deviceset="DEVBOARD_ESP8266_NODEMCU_V3" device="DEVBOARD" package3d_urn="urn:adsk.eagle:package:36294322/5"/>
 <part name="R5" library="OPL_Resistor" library_urn="urn:adsk.eagle:library:8004883" deviceset="SMD-RES-68R-1%-1/10W(0603)" device="" package3d_urn="urn:adsk.eagle:package:8004941/1" value="68 OHM"/>
 <part name="SUPPLY6" library="supply2" library_urn="urn:adsk.eagle:library:372" deviceset="GND" device=""/>
@@
 <part name="POWER" library="CustomParts-Josh" library_urn="urn:adsk.eagle:library:21718240" deviceset="CONN-WR-TBL-2POS" device="" package3d_urn="urn:adsk.eagle:package:36293342/3" value=" 691103110003 "/>
 <part name="ADD-ON" library="JST XH Connectors" deviceset="JST-XH-06-PIN" device="-VERT-ROUND-PAD"/>
-<part name="MOTION" library="JST XH Connectors" deviceset="JST-XH-03-PIN" device="-VERT-ROUND-PAD"/>
+<part name="PIR.SENSOR" library="JST XH Connectors" deviceset="JST-XH-03-PIN" device="-VERT-ROUND-PAD"/>
 <part name="SUPPLY3" library="supply2" library_urn="urn:adsk.eagle:library:372" deviceset="GND" device=""/>
 <part name="H1" library="holes" library_urn="urn:adsk.eagle:library:237" deviceset="MOUNT-PAD-ROUND" device="3.2" package3d_urn="urn:adsk.eagle:package:14282/1"/>
@@
 <part name="H3" library="holes" library_urn="urn:adsk.eagle:library:237" deviceset="MOUNT-PAD-ROUND" device="3.2" package3d_urn="urn:adsk.eagle:package:14282/1" value="MOUNT-PAD"/>
 <part name="H4" library="holes" library_urn="urn:adsk.eagle:library:237" deviceset="MOUNT-PAD-ROUND" device="3.2" package3d_urn="urn:adsk.eagle:package:14282/1"/>
-<part name="IC4" library="CustomParts-Josh" library_urn="urn:adsk.eagle:library:21718240" deviceset="LM2596" device="S" package3d_urn="urn:adsk.eagle:package:16438/2"/>
+<part name="IC4" library="CustomParts-Josh" library_urn="urn:adsk.eagle:library:21718240" deviceset="LM2596" device="S" package3d_urn="urn:adsk.eagle:package:37231383/1"/>
 <part name="CT3" library="Capacitor" library_urn="urn:adsk.eagle:library:16290819" deviceset="C-POL-US" device="ECAP-8.5MM" package3d_urn="urn:adsk.eagle:package:16290889/1" technology="_" value="220UF"/>
 <part name="CT4" library="Capacitor" library_urn="urn:adsk.eagle:library:16290819" deviceset="C-POL-US" device="ECAP-8.5MM" package3d_urn="urn:adsk.eagle:package:16290889/1" technology="_" value="220UF"/>
@@
 <attribute name="VALUE" x="4.953" y="41.275" size="1.778" layer="96" align="bottom-center"/>
 </instance>
-<instance part="5V_LED" gate="G$1" x="27.94" y="12.7" smashed="yes" rot="R90">
-<attribute name="NAME" x="27.94" y="8.001" size="1.778" layer="95" align="top-center"/>
-<attribute name="WS2811" x="27.94" y="12.7" size="1.778" layer="96" rot="R90"/>
+<instance part="5V_LED" gate="G$1" x="27.94" y="12.7" smashed="yes" rot="MR270">
+<attribute name="NAME" x="27.94" y="17.399" size="1.778" layer="95" rot="MR180" align="top-center"/>
+<attribute name="WS2811" x="27.94" y="12.7" size="1.778" layer="96" rot="MR270"/>
 </instance>
 <instance part="SUPPLY14" gate="GND" x="35.56" y="5.08" smashed="yes"/>
@@
 <attribute name="VALUE" x="51.435" y="60.325" size="1.778" layer="96"/>
 </instance>
-<instance part="POWER" gate="G$1" x="-7.62" y="30.48" smashed="yes" rot="R90">
-<attribute name="NAME" x="-6.698" y="26.87" size="1.016" layer="95" rot="R90" align="bottom-right"/>
-<attribute name="VALUE" x="-5.04" y="26.92" size="1.016" layer="96" rot="R90" align="bottom-right"/>
+<instance part="POWER" gate="G$1" x="-7.62" y="33.02" smashed="yes" rot="MR270">
+<attribute name="NAME" x="-6.698" y="36.63" size="1.016" layer="95" rot="MR270" align="bottom-right"/>
+<attribute name="VALUE" x="-5.04" y="36.58" size="1.016" layer="96" rot="MR270" align="bottom-right"/>
 </instance>
 <instance part="ADD-ON" gate="-1" x="83.82" y="38.1" smashed="yes" rot="MR0">
@@
 <attribute name="NAME" x="81.28" y="24.638" size="1.524" layer="95" rot="MR0"/>
 </instance>
-<instance part="MOTION" gate="-1" x="83.82" y="10.16" smashed="yes" rot="R180">
+<instance part="PIR.SENSOR" gate="-1" x="83.82" y="10.16" smashed="yes" rot="R180">
 <attribute name="NAME" x="81.28" y="10.922" size="1.524" layer="95" rot="R180"/>
 </instance>
-<instance part="MOTION" gate="-2" x="83.82" y="12.7" smashed="yes" rot="R180">
+<instance part="PIR.SENSOR" gate="-2" x="83.82" y="12.7" smashed="yes" rot="R180">
 <attribute name="NAME" x="81.28" y="13.462" size="1.524" layer="95" rot="R180"/>
 </instance>
-<instance part="MOTION" gate="-3" x="83.82" y="15.24" smashed="yes" rot="R180">
+<instance part="PIR.SENSOR" gate="-3" x="83.82" y="15.24" smashed="yes" rot="R180">
 <attribute name="NAME" x="81.28" y="16.002" size="1.524" layer="95" rot="R180"/>
 </instance>
@@
 <wire x1="88.9" y1="7.62" x2="88.9" y2="10.16" width="0.1524" layer="91"/>
 <wire x1="88.9" y1="10.16" x2="86.36" y2="10.16" width="0.1524" layer="91"/>
-<pinref part="MOTION" gate="-1" pin="S"/>
+<pinref part="PIR.SENSOR" gate="-1" pin="S"/>
 </segment>
 <segment>
 <pinref part="SUPPLY6" gate="GND" pin="GND"/>
 <wire x1="0" y1="30.48" x2="0" y2="27.94" width="0.1524" layer="91"/>
-<pinref part="POWER" gate="G$1" pin="1"/>
-<wire x1="0" y1="30.48" x2="-2.54" y2="30.48" width="0.1524" layer="91"/>
+<pinref part="POWER" gate="G$1" pin="2"/>
+<wire x1="-2.54" y1="30.48" x2="0" y2="30.48" width="0.1524" layer="91"/>
 </segment>
 <segment>
@@
 </segment>
 <segment>
-<pinref part="5V_LED" gate="G$1" pin="1"/>
 <pinref part="SUPPLY14" gate="GND" pin="GND"/>
+<wire x1="35.56" y1="10.16" x2="35.56" y2="7.62" width="0.1524" layer="91"/>
+<pinref part="5V_LED" gate="G$1" pin="3"/>
 <wire x1="33.02" y1="10.16" x2="35.56" y2="10.16" width="0.1524" layer="91"/>
-<wire x1="35.56" y1="10.16" x2="35.56" y2="7.62" width="0.1524" layer="91"/>
 </segment>
 <segment>
@@
 <pinref part="SUPPLY25" gate="G$1" pin="5V"/>
 <wire x1="93.98" y1="15.24" x2="93.98" y2="17.78" width="0.1524" layer="91"/>
-<pinref part="MOTION" gate="-3" pin="S"/>
-</segment>
-<segment>
-<pinref part="5V_LED" gate="G$1" pin="3"/>
+<pinref part="PIR.SENSOR" gate="-3" pin="S"/>
+</segment>
+<segment>
 <pinref part="SUPPLY16" gate="G$1" pin="5V"/>
+<wire x1="35.56" y1="15.24" x2="35.56" y2="17.78" width="0.1524" layer="91"/>
+<pinref part="5V_LED" gate="G$1" pin="1"/>
 <wire x1="33.02" y1="15.24" x2="35.56" y2="15.24" width="0.1524" layer="91"/>
-<wire x1="35.56" y1="15.24" x2="35.56" y2="17.78" width="0.1524" layer="91"/>
-</segment>
-<segment>
-<pinref part="U$1" gate="G$1" pin="VV"/>
-<wire x1="-88.9" y1="83.82" x2="-101.6" y2="83.82" width="0.1524" layer="91"/>
-<label x="-101.6" y="83.82" size="1.778" layer="95" rot="R180" xref="yes"/>
 </segment>
 <segment>
@@
 <junction x="53.34" y="91.44"/>
 </segment>
+<segment>
+<pinref part="U$1" gate="G$1" pin="VIN"/>
+<wire x1="-78.74" y1="109.22" x2="-78.74" y2="114.3" width="0.1524" layer="91"/>
+<label x="-78.74" y="114.3" size="1.27" layer="95" rot="R90" xref="yes"/>
+</segment>
 </net>
 <net name="N$12" class="2">
@@
 <label x="96.52" y="12.7" size="1.778" layer="95" xref="yes"/>
 <wire x1="86.36" y1="12.7" x2="96.52" y2="12.7" width="0.1524" layer="91"/>
-<pinref part="MOTION" gate="-2" pin="S"/>
+<pinref part="PIR.SENSOR" gate="-2" pin="S"/>
 </segment>
 <segment>
@@
 <wire x1="5.08" y1="33.02" x2="5.08" y2="35.56" width="0.1524" layer="91"/>
 <pinref part="SUPPLY5" gate="G$1" pin="12V"/>
-<pinref part="POWER" gate="G$1" pin="2"/>
-<wire x1="5.08" y1="33.02" x2="-2.54" y2="33.02" width="0.1524" layer="91"/>
+<pinref part="POWER" gate="G$1" pin="1"/>
+<wire x1="-2.54" y1="33.02" x2="5.08" y2="33.02" width="0.1524" layer="91"/>
 </segment>
 <segment>
@@
 <net name="WS2812_DATA" class="2">
 <segment>
+<label x="38.1" y="12.7" size="1.778" layer="95" xref="yes"/>
 <pinref part="5V_LED" gate="G$1" pin="2"/>
 <wire x1="33.02" y1="12.7" x2="38.1" y2="12.7" width="0.1524" layer="91"/>
-<label x="38.1" y="12.7" size="1.778" layer="95" xref="yes"/>
 </segment>
 <segment>
@@
 </segment>
 </net>
-<net name="3.3V" class="1">
+<net name="VCC_3V3.2" class="1">
 <segment>
 <label x="91.44" y="35.56" size="1.27" layer="95" xref="yes"/>
@@
 </segment>
 </net>
+<net name="VCC_3V3.1" class="0">
+<segment>
+<pinref part="U$1" gate="G$1" pin="3.3V@2"/>
+<wire x1="-71.12" y1="109.22" x2="-71.12" y2="114.3" width="0.1524" layer="91"/>
+<label x="-71.12" y="114.3" size="1.27" layer="95" rot="R90" xref="yes"/>
+</segment>
+</net>
+<net name="VCC_3V3.3" class="0">
+<segment>
+<pinref part="U$1" gate="G$1" pin="3.3V@5"/>
+<wire x1="-60.96" y1="109.22" x2="-60.96" y2="114.3" width="0.1524" layer="91"/>
+<label x="-60.96" y="114.3" size="1.27" layer="95" rot="R90" xref="yes"/>
+</segment>
+</net>
